File: traffic_light_s2_timer.kicad_sch (KiCad schematic)
At the start: 23 parts, among them SW1 方案SW, SW2 调试LOAD, U11 74LS160 南北个位, U12 74LS160 南北十位, U13 74LS160 东西个位, U14 74LS160 东西十位, U21 74LS157 南北个位2选1, U22 74LS157 南北十位一级, U22p 74LS157 南北十位二级, U23 74LS157 东西个位2选1, U24 74LS157 东西十位一级, U24p 74LS157 东西十位二级, U31 74LS283 南北个位补码, U32 74LS283 南北十位补码, U33 74LS283 东西个位补码, U34 74LS283 东西十位补码, U35 74LS32 ROLE, U41 74LS04, U42 74LS04, U43 74LS04, U44 74LS04

Commit message: feat: Generate KiCad SPICE Circuit Schematic
Co-authored-by: traeagent <traeagent@users.noreply.github.com>
Parts:
- removed U22p: 74LS157 南北十位二级, symbol TrafficLight:74LS157
- removed U24p: 74LS157 东西十位二级, symbol TrafficLight:74LS157
- removed unit 5 of U41
- added U22P: 74LS157 南北十位二级, symbol TrafficLight:74LS157
- added U24P: 74LS157 东西十位二级, symbol TrafficLight:74LS157
- added U45: 74LS04 方案取反, symbol TrafficLight:74LS04
- SW1: value 方案SW -> 方案选择
- SW2: value 调试LOAD -> 调试装载
- U21: value 74LS157 南北个位2选1 -> 74LS157 南北个位装载
- U23: value 74LS157 东西个位2选1 -> 74LS157 东西个位装载
- U35: value 74LS32 ROLE -> 74LS32 ROLE合成
- U41: value 74LS04 -> 74LS04 南北个位取反
- U42: value 74LS04 -> 74LS04 南北十位取反
- U43: value 74LS04 -> 74LS04 东西个位取反
- U44: value 74LS04 -> 74LS04 东西十位取反
Connections:
- net NS_UNI_2 is gone; now on net GND: U21.12 (4Y)
- net +5V: now also U11.2 (CLK), U11.9 (~{LOAD}), U13.2 (CLK), U13.9 (~{LOAD}), U21.10 (3B), U21.15 (~{G}), U21.2 (1A), U22.10 (3B), U22.11 (3A), U22.15 (~{G}), U22.2 (1A), U22.5 (2A), U22P.16 (+5V), U22P.3 (1B), U22P.6 (2B), U24P.10 (3B), U24P.16 (+5V), U24P.3 (1B), U24P.6 (2B), U45.14 (+5V); no longer C_POR.2, U11.8 (GND), U12.8 (GND), U13.8 (GND), U14.8 (GND), U21.8 (GND), U22.8 (GND), U23.1 (S), U23.11 (3A), U23.12 (4Y), U23.14 (4A), U23.3 (1B), U23.6 (2B), U23.8 (GND), U24.1 (S), U24.11 (3A), U24.14 (4A), U24.3 (1B), U24.8 (GND), U31.13 (GND), U32.13 (GND), U33.13 (GND), U34.13 (GND), U35.2 (B), U35.7 (GND), U41.7 (GND), U42.7 (GND), U43.7 (GND), U44.7 (GND)
- net CLK_GATED: now also U11.10 (ENT), U12.10 (ENT)
- net NSW: now also U45.2 (Y)
- net PH_EW: now also U24P.13 (4B)
- net PH_NS: now also U22P.13 (4B)
- net SW: now also U24.11 (3A), U22P.10 (3B), U45.1 (A); no longer U24.6 (2B)
- net GND: now reaches U21.1 (S)
- net GND: now also R_POR.2, U11.8 (GND), U12.8 (GND), U13.8 (GND), U14.8 (GND), U21.11 (3A), U21.14 (4A), U21.3 (1B), U21.6 (2B), U21.8 (GND), U22.1 (S), U22.14 (4A), U22.3 (1B), U22.6 (2B), U22.8 (GND), U23.1 (S), U23.11 (3A), U23.12 (4Y), U23.14 (4A), U23.3 (1B), U23.6 (2B), U23.8 (GND), U24.1 (S), U24.14 (4A), U24.3 (1B), U24.6 (2B), U24.8 (GND), U31.13 (GND), U32.13 (GND), U33.13 (GND), U34.13 (GND), U35.7 (GND), U41.7 (GND), U42.7 (GND), U43.7 (GND), U44.7 (GND), U22P.12 (4Y), U22P.14 (4A), U22P.15 (~{G}), U22P.8 (GND), U24P.12 (4Y), U24P.14 (4A), U24P.15 (~{G}), U24P.8 (GND), U45.7 (GND)
- net at U11.11 (QD): now also U41.9 (A)
- net CARRY_NS: now reaches U11.13 (QB)
- net CARRY_NS: now also U12.2 (CLK), U12.9 (~{LOAD})
- net at U11.15 (RCO): now also U41.3 (A)
- net LOAD_NS: now reaches U11.7 (ENP)
- net LOAD_NS: now also C_POR.2, R_POR.1, U12.13 (QB), U12.7 (ENP), U35.2 (B)
- net at U12.11 (QD): now also U42.9 (A)
- net at U12.15 (RCO): now also U42.3 (A)
- net at U41.8 (Y): now also U31.1 (A4)
- net at U42.8 (Y): now also U32.1 (A4)
- net NS_BCD_UNI_3: now reaches U31.15 (S4)
- net NS_BCD_TEN_3: now reaches U32.15 (S4)
- net CARRY_EW: now reaches U13.13 (QB)
- net CARRY_EW: now also U14.2 (CLK), U14.9 (~{LOAD})
- net EW_BCD_UNI_3: now reaches U33.15 (S4)
- net EW_BCD_TEN_3: now reaches U34.15 (S4)
- net EWNTEN_0: no longer names the net of U44.2 (Y)
- net EWNTEN_1: no longer names the net of U44.4 (Y)
- net EWNTEN_2: no longer names the net of U44.6 (Y)
- net EWNTEN_3: no longer names the net of U34.1 (A4), U44.8 (Y)
- net EWNUNI_0: no longer names the net of U43.2 (Y)
- net EWNUNI_1: no longer names the net of U43.4 (Y)
- net EWNUNI_2: no longer names the net of U43.6 (Y)
- net EWNUNI_3: no longer names the net of U33.1 (A4), U43.8 (Y)
- net EWT1_2: no longer names the net of U24.12 (4Y)
- net EWT1_2: now also U24P.2 (1A)
- net EWT1_3: no longer names the net of U24.9 (3Y)
- net EWT1_3: now also U24P.1 (S)
- net EW_CNT_TEN_0: no longer names the net of U44.1 (A)
- net EW_CNT_TEN_1: no longer names the net of U14.15 (RCO), U44.3 (A)
- net EW_CNT_TEN_2: no longer names the net of U44.5 (A)
- net EW_CNT_TEN_3: no longer names the net of U14.11 (QD), U44.9 (A)
- net EW_CNT_UNI_0: no longer names the net of U43.1 (A)
- net EW_CNT_UNI_1: no longer names the net of U13.15 (RCO), U43.3 (A)
- net EW_CNT_UNI_2: no longer names the net of U43.5 (A)
- net EW_CNT_UNI_3: no longer names the net of U13.11 (QD), U43.9 (A)
- net EW_UNI_3: no longer names the net of U23.9 (3Y)
- net NS_UNI_3: no longer names the net of U21.9 (3Y)
- net TNS1_2: no longer names the net of U22.12 (4Y)
- net TNS1_2: now also U22P.2 (1A)
- net TNS1_3: no longer names the net of U22.9 (3Y)
- net TNS1_3: now also U22P.1 (S)
- no-connect marks 8 -> 6
Other:
- note added: "283: A=计数位取反, B=1010 固定, S=9-N 倒计时显示总线 -> 第5节 74LS48"
- note added: "SW: 方案位(SW=0 二: 30/3/20/3s, SW=1 一: 20/5/20/5s) | SW2: 调试手动装载 | POR: 上电微分脉冲强制装载"
- note added: "东西轴(下): 绿79/黄96/休66 (SW=0) | 十位二级 A组=绿十位(东西固定7, 南北=SW) | 休十位: 南北固定7, 东西=SW"
- note added: "南北轴(上): 绿69/黄96/休76 (SW=0方案二) | 装载值=99-显示初值 | 计满99 -> RCO=LOAD 同步装载 | 两轴恒计数"
- note added: "第2节 计时电路 —— 74LS157x6 装载网络 + 74LS160x4 计数链 + 74LS04x8 取反 + 74LS283x4 九进制补码(显示值=9-计数值)"
- note added: "计数链: CLK=CLK_GATED | 个位 ENP/ENT=+5V 恒计数, RCO=CARRY -> 十位 ENP/ENT | 十位 RCO=LOAD 反馈两片同步装载"
- note removed: "SW位: 南北绿十位 1A=SW(6/7)、黄休个位 2B=(NSW)(6/4); 东西休十位 U24 1B=SW(6/7)、黄休个位 U23 2B=NSW"
- note removed: "上电复位: VCC->C_POR(10uF)->LOAD_NS 微分窄脉冲强制装载, R_POR(1k)下拉 (东西轴建议同样加一组)"
- note removed: "东西轴对称: U23/U24/U24P 装载网络, U13/U14 计数链, U33/U34 补码; LOAD_EW=U14 RCO"
- note removed: "南北轴装载网络: U21个位(绿9固定/黄休6/4) U22十位一级(T0选黄9, T1选休7) U22P十位二级(PH_NS选绿十位SW)"
- note removed: "南北轴计数链+补码: U11/U12 从装载值计到99, RCO=LOAD_NS 同步装载; 非门取反 -> U31/U32 +1010 -> 9-N 显示值"
